Commit message: fix: fixed joint axis

File: op3_description/urdf/robotis_op3.structure.head.xacro (robot description, xacro)
@@ -33,5 +33,5 @@
     <child link="head_tilt_link"/>
     <origin xyz="0.010 0.019 0.0285" rpy="0 0 0" />
-    <axis xyz="0 -1 0" />
+    <axis xyz="0 1 0" />
     <limit effort="1000" velocity="100" lower="${-pi*0.9}" upper="${pi*0.9}" />
     <dynamics damping="0.1" friction="0.0" />

File: op3_description/urdf/robotis_op3.structure.larm.xacro (robot description, xacro)
@@ -33,5 +33,5 @@
     <child link="l_sho_roll_link"/>
     <origin xyz="0.019 0.0285 -0.010" rpy="0 0 0" />
-    <axis xyz="-1 0 0" />
+    <axis xyz="1 0 0" />
     <limit effort="1000" velocity="100" lower="${-pi*0.9}" upper="${pi*0.9}" />
     <dynamics damping="0.1" friction="0.0" />

File: op3_description/urdf/robotis_op3.structure.lleg.xacro (robot description, xacro)
@@ -11,5 +11,5 @@
     <child link="l_hip_yaw_link"/>
     <origin xyz="0.0 0.035 0.0" rpy="0 0 0" />
-    <axis xyz="0 0 -1" />
+    <axis xyz="0 0 1" />
     <limit effort="1000" velocity="100" lower="${-pi*0.9}" upper="${pi*0.9}" />
     <dynamics damping="0.1" friction="0.0" />
@@ -33,5 +33,5 @@
     <child link="l_hip_roll_link"/>
     <origin xyz="-0.024 0.0 -0.0285" rpy="0 0 0" />
-    <axis xyz="-1 0 0" />
+    <axis xyz="1 0 0" />
     <limit effort="1000" velocity="100" lower="${-pi*0.9}" upper="${pi*0.9}" />
     <dynamics damping="0.1" friction="0.0" />
@@ -99,5 +99,5 @@
     <child link="l_ank_pitch_link"/>
     <origin xyz="0 0 -0.110" rpy="0 0 0" />
-    <axis xyz="0 -1 0" />
+    <axis xyz="0 1 0" />
     <limit effort="1000" velocity="100" lower="${-pi*0.9}" upper="${pi*0.9}" />
     <dynamics damping="0.1" friction="0.0" />

File: op3_description/urdf/robotis_op3.structure.rarm.xacro (robot description, xacro)
@@ -33,5 +33,5 @@
     <child link="r_sho_roll_link"/>
     <origin xyz="0.019 -0.0285 -0.010" rpy="0 0 0" />
-    <axis xyz="-1 0 0" />
+    <axis xyz="1 0 0" />
     <limit effort="1000" velocity="100" lower="${-pi*0.9}" upper="${pi*0.9}" />
     <dynamics damping="0.1" friction="0.0" />

File: op3_description/urdf/robotis_op3.structure.rleg.xacro (robot description, xacro)
@@ -11,5 +11,5 @@
     <child link="r_hip_yaw_link"/>
     <origin xyz="0.0 -0.035 0.0" rpy="0 0 0" />
-    <axis xyz="0 0 -1" />
+    <axis xyz="0 0 1" />
     <limit effort="1000" velocity="100" lower="${-pi*0.9}" upper="${pi*0.9}" />
     <dynamics damping="0.1" friction="0.0" />
@@ -33,5 +33,5 @@
     <child link="r_hip_roll_link"/>
     <origin xyz="-0.024 0.0 -0.0285" rpy="0 0 0" />
-    <axis xyz="-1 0 0" />
+    <axis xyz="1 0 0" />
     <limit effort="1000" velocity="100" lower="${-pi*0.9}" upper="${pi*0.9}" />
     <dynamics damping="0.1" friction="0.0" />
@@ -55,5 +55,5 @@
     <child link="r_hip_pitch_link"/>
     <origin xyz="0.0241 -0.019 0.0" rpy="0 0 0" />
-    <axis xyz="0 -1 0" />
+    <axis xyz="0 1 0" />
     <limit effort="1000" velocity="100" lower="${-pi*0.9}" upper="${pi*0.9}" />
     <dynamics damping="0.1" friction="0.0" />
@@ -77,5 +77,5 @@
     <child link="r_knee_link"/>
     <origin xyz="0.0 0.0 -0.11015" rpy="0 0 0" />
-    <axis xyz="0 -1 0" />
+    <axis xyz="0 1 0" />
     <limit effort="1000" velocity="100" lower="${-pi*0.9}" upper="${pi*0.9}" />
     <dynamics damping="0.1" friction="0.0" />
